Commit message: update controller to by pose

File: src/robot/urdf/robot.urdf (robot description, URDF)
Before this commit: robot robot, 12 links, 11 joints
Links:
- removed link Gap_base
- removed link Gap_motor
- removed link left_finger
- removed link right_finger
- added link gripper_left, mass 0.0029678; collision mesh filename=package://my_arm_robot/meshes/gripper_left.STL; visual mesh filename=package://my_arm_robot/meshes/gripper_left.STL
- added link gripper_right, mass 0.0029678; collision mesh filename=package://my_arm_robot/meshes/gripper_right.STL; visual mesh filename=package://my_arm_robot/meshes/gripper_right.STL
- added link tool_center_point
- link Link_1: mass 0.29405 -> 0.35373
- link Link_2: mass 0.56692 -> 0.32748
- link Link_3: mass 0.28134 -> 0.64467
- link Link_4: mass 0.24763 -> 0.35757
- link Link_5: mass 0.24762 -> 0.21575
- link Link_6: mass 0.13168 -> 0.025118
- link base_link: mass 0.35438 -> 0.467996
Joints:
- removed joint Gap_base_joint
- removed joint gripper_motor_joint
- removed joint left_finger_joint
- removed joint right_finger_joint
- added joint gripper_left_joint: type revolute, parent Link_6, child gripper_left, origin xyz=0.032692 -0.015993 0.061756 rpy=1.5708 -1.1863 2.2467, axis 0 0 1, limit lower=-1.57 upper=1.57 effort=20 velocity=1, mimic joint=gripper_right_joint multiplier=-1 offset=0
- added joint gripper_right_joint: type revolute, parent Link_6, child gripper_right, origin xyz=-0.008556 0.035448 0.061693 rpy=-1.5708 -1.1863 -0.89493, axis 0 0 1, limit lower=-1.57 upper=1.57 effort=20 velocity=1
- added joint tcp_joint: type fixed, parent Link_6, child tool_center_point, origin xyz=0 0 0.15 rpy=0 0 0
- joint Link_1_joint: limit lower=-3.14 upper=3.14 effort=100 velocity=0 -> lower=-1.57 upper=1.57 effort=100 velocity=1; origin xyz=0 0 0.109 rpy=0 0 0 -> xyz=0 0 0.1214 rpy=0 0 0
- joint Link_2_joint: axis 0 0 -1 -> 0 0 1; limit lower=-1.57 upper=1.57 effort=100 velocity=0 -> lower=-1.57 upper=1.57 effort=100 velocity=1; origin xyz=0 -0.0715 0.0645 rpy=1.5708 -1.5708 0 -> xyz=-0.037236 0.040478 0.046 rpy=1.5708 -1.5643 -2.3979
- joint Link_3_joint: axis 0 0 1 -> 0 0 -1; limit lower=-2.5 upper=2.5 effort=100 velocity=0 -> lower=-1.57 upper=1.57 effort=100 velocity=1; origin xyz=0.10408 -0.10802 0 rpy=-3.1416 0 -1.5708 -> xyz=0.11 0 0 rpy=3.1416 0 1.5773
- joint Link_4_joint: limit lower=-3.14 upper=3.14 effort=100 velocity=0 -> lower=-1.57 upper=1.57 effort=100 velocity=1; origin xyz=0.14857 -0.020684 0 rpy=3.1416 0 0 -> xyz=-0.070463 0.12975 0.055 rpy=-1.5708 0 0.003562
- joint Link_5_joint: limit lower=-2 upper=2 effort=100 velocity=0 -> lower=-1.57 upper=1.57 effort=100 velocity=1; origin xyz=0.071006 -0.008387 0.047 rpy=-1.5708 0.23999 -1.6884 -> xyz=0.003472 -0.040251 0.056 rpy=1.5708 0.0035488 0.086047
- joint Link_6_joint: axis 0 0 -1 -> 0 0 1; limit lower=-3.14 upper=3.14 effort=100 velocity=0 -> lower=-1.57 upper=1.57 effort=100 velocity=1; origin xyz=0.0715 0 0.047 rpy=1.5708 -0.54029 1.5708 -> xyz=-0.00059549 0.085198 -0.041 rpy=-1.5708 -0.82976 0.0069894

Commit message: update kinematic

File: src/robot/urdf/robot.urdf (robot description, URDF)
Before this commit: robot robot, 11 links, 10 joints
Links:
- removed link gripper_left
- removed link gripper_right
- removed link world
- added link Base_Gap, mass 0.02487; collision mesh filename=package://my_arm_robot/meshes/Base_Gap.STL; visual mesh filename=package://my_arm_robot/meshes/Base_Gap.STL
- added link finger_left, mass 0.0029678; collision mesh filename=package://my_arm_robot/meshes/finger_left.STL; visual mesh filename=package://my_arm_robot/meshes/finger_left.STL
- added link finger_right, mass 0.0029678; collision mesh filename=package://my_arm_robot/meshes/finger_right.STL; visual mesh filename=package://my_arm_robot/meshes/finger_right.STL
- link Link_5: mass 0.21575 -> 0.18274
- link Link_6: mass 0.025118 -> 0.033013
- link base_link: mass 0.467996 -> 0.467996005301711
Joints:
- removed joint gripper_left_joint
- removed joint gripper_right_joint
- removed joint world_joint
- added joint Base_Gap_joint: type fixed, parent Link_6, child Base_Gap, origin xyz=0 0 0.008 rpy=0 0 1.6175, axis 0 0 0
- added joint finger_left_joint: type revolute, parent Base_Gap, child finger_left, origin xyz=0.0155 -0.032928 0.054756 rpy=1.5708 -1.1863 1.5708, axis 0 0 -1, limit lower=-1.57 upper=1.57 effort=50 velocity=1, mimic joint=finger_right_joint multiplier=-1 offset=0
- added joint finger_right_joint: type revolute, parent Base_Gap, child finger_right, origin xyz=0.0155 0.033007 0.054693 rpy=-1.5708 -1.1863 -1.5708, axis 0 0 -1, limit lower=-1.57 upper=1.57 effort=50 velocity=1
- joint Link_1_joint: axis 0 0 1 -> 0 0 -1; limit lower=-1.57 upper=1.57 effort=100 velocity=1 -> lower=-1.57 upper=1.57 effort=100 velocity=2; origin xyz=0 0 0.1214 rpy=0 0 0 -> xyz=0 0 0.122 rpy=0 0 0
- joint Link_2_joint: axis 0 0 1 -> 0 0 -1; limit lower=-1.57 upper=1.57 effort=100 velocity=1 -> lower=-1.57 upper=1.57 effort=100 velocity=2; origin xyz=-0.037236 0.040478 0.046 rpy=1.5708 -1.5643 -2.3979 -> xyz=0.0047777 -0.054792 0.046 rpy=1.5708 -0.75408 0.086978
- joint Link_3_joint: axis 0 0 -1 -> 0 0 1; limit lower=-1.57 upper=1.57 effort=100 velocity=1 -> lower=-1.57 upper=1.57 effort=100 velocity=2; origin xyz=0.11 0 0 rpy=3.1416 0 1.5773 -> xyz=0.11 0 0 rpy=3.1416 0 -0.75408
- joint Link_4_joint: limit lower=-1.57 upper=1.57 effort=100 velocity=1 -> lower=-1.57 upper=1.57 effort=50 velocity=2; origin xyz=-0.070463 0.12975 0.055 rpy=-1.5708 0 0.003562 -> xyz=0.057193 -0.043058 0.055 rpy=-1.5708 0.13232 -0.85642
- joint Link_5_joint: limit lower=-1.57 upper=1.57 effort=100 velocity=1 -> lower=-1.57 upper=1.57 effort=50 velocity=2; origin xyz=0.003472 -0.040251 0.056 rpy=1.5708 0.0035488 0.086047 -> xyz=-0.00094211 0.04299 0.056 rpy=1.5708 -1.2184 -3.1197
- joint Link_6_joint: axis 0 0 1 -> 0 0 -1; limit lower=-1.57 upper=1.57 effort=100 velocity=1 -> lower=-1.57 upper=1.57 effort=50 velocity=2; origin xyz=-0.00059549 0.085198 -0.041 rpy=-1.5708 -0.82976 0.0069894 -> xyz=0.084 0 -0.043 rpy=1.5708 0.016437 1.5708
- joint tcp_joint: origin xyz=0 0 0.15 rpy=0 0 0 -> xyz=0 0 0.1 rpy=0 0 0

Commit message: init newton raphson

File: src/robot/urdf/robot.urdf (robot description, URDF)
Before this commit: robot robot, 11 links, 10 joints
Joints:
- removed joint finger_left_joint
- removed joint finger_right_joint
- added joint gripper_left_joint: type revolute, parent Base_Gap, child finger_left, origin xyz=0.0155 -0.032928 0.054756 rpy=1.5708 -1.1863 1.5708, axis 0 0 -1, limit lower=-1.57 upper=1.57 effort=50 velocity=1, mimic joint=gripper_right_joint multiplier=-1 offset=0
- added joint gripper_right_joint: type revolute, parent Base_Gap, child finger_right, origin xyz=0.0155 0.033007 0.054693 rpy=-1.5708 -1.1863 -1.5708, axis 0 0 -1, limit lower=-1.57 upper=1.57 effort=50 velocity=1
